Commit message: Update real robot setup data at 3-412

File: src/coop_assembly/data/models/kuka_kr6_r900/urdf/mit_3-412_workspace.urdf (robot description, URDF)
Before this commit: robot mit_3-412_workspace, 9 links, 8 joints
Joints:
- joint workspace_baselink_to_print_table: origin xyz=0.7 0 0.0 rpy=0 0 0 -> xyz=0.7 0 -16.23 rpy=0 0 0
